File: Boards/Toolhead Board/toolhead_board.kicad_sch (KiCad schematic)
At the start: 29 parts, among them J1 Molex 502386-0470, J10 Molex 502386-0370, J2 Molex 213228-1810, J3 Molex 502386-0370, J4 Molex 502386-0370, J5 Conn_02x04_Odd_Even, J6 Molex 502386-0470, J7 Molex 502386-0270, J8 Molex 502386-0370, J9 Molex 43650-0210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

Commit message: 4 layer board
Parts:
- added J11: Molex 502386-0270, Connector_Molex:Molex_CLIK-Mate_502386-0270_1x02-1MP_P1.25mm_Horizontal, symbol Connector_Generic:Conn_01x02
- added J12: Conn_02x02_Odd_Even, Connector_PinHeader_2.00mm:PinHeader_2x02_P2.00mm_Vertical, symbol Connector_Generic:Conn_02x02_Odd_Even
- J1: value Molex 502386-0470 -> Molex 502382-0470; footprint Connector_Molex:Molex_CLIK-Mate_502386-0470_1x04-1MP_P1.25mm_Horizontal -> Connector_Molex:Molex_CLIK-Mate_502382-0470_1x04-1MP_P1.25mm_Vertical
Connections:
- net +5V: now also J2.3 (Pin_3); no longer J2.4 (Pin_4)
- net DATA+: now also J2.14 (Pin_14); no longer J2.21 (Pin_21)
- net GND: now also J2.4 (Pin_4); no longer J2.5 (Pin_5), J2.6 (Pin_6)
- net GNDA: now also J2.18 (Pin_18), J11.2 (Pin_2); no longer J2.22 (Pin_22)
- net HE_FAN_GND: now also J2.6 (Pin_6); no longer J2.16 (Pin_16)
- net HE_FAN_TACH: now also J2.8 (Pin_8); no longer J2.13 (Pin_13)
- net MOTOR_1A: now also J1.1 (Pin_1), J2.19 (Pin_19); no longer J1.4 (Pin_4), J2.7 (Pin_7)
- net MOTOR_1B: now also J1.2 (Pin_2), J2.20 (Pin_20); no longer J1.3 (Pin_3), J2.8 (Pin_8)
- net MOTOR_2A: now also J1.3 (Pin_3), J2.21 (Pin_21); no longer J1.2 (Pin_2), J2.9 (Pin_9)
- net MOTOR_2B: now also J1.4 (Pin_4), J2.22 (Pin_22); no longer J1.1 (Pin_1), J2.10 (Pin_10)
- net PC_FAN0_TACH: now also J2.9 (Pin_9); no longer J2.14 (Pin_14)
- net PC_FAN1_TACH: now also J2.10 (Pin_10); no longer J2.15 (Pin_15)
- net PC_FAN_GND: now also J10.1 (Pin_1), J2.7 (Pin_7); no longer J10.3 (Pin_3), J2.17 (Pin_17)
- net PC_FAN_PWR: now also J10.3 (Pin_3); no longer J10.1 (Pin_1)
- net RGB: now also J2.17 (Pin_17); no longer J2.12 (Pin_12)
- net SCK+: now also J2.11 (Pin_11); no longer J2.18 (Pin_18)
- net SCK-: now also J2.12 (Pin_12); no longer J2.19 (Pin_19)
- net TH0: now also J2.16 (Pin_16); no longer J2.11 (Pin_11)
- net at L1.1: now also J12.4 (Pin_4); no longer J6.1 (Pin_1)
- net at L4.1: now also J6.4 (Pin_4); no longer J6.3 (Pin_3)
- net at L3.1: now also J6.3 (Pin_3); no longer J6.4 (Pin_4)
- net DATA- renamed DATA-/Z_END
- net DATA-/Z_END: now also J2.13 (Pin_13), J12.2 (Pin_2); no longer J2.20 (Pin_20)
- net HE0 renamed HE_GND
- net HE_GND: now also J2.5 (Pin_5); no longer J2.3 (Pin_3)
- new net: J12.1 (Pin_1), J12.3 (Pin_3), J6.1 (Pin_1)
- new net XEND: J11.1 (Pin_1), J2.15 (Pin_15)
Other:
- note added: "Gauge Enable"
- note added: "X Endstop"
- note added: "or Z Endstop"
- moved on the sheet: J10, J6, J9
